Commit message: add urdf python code and change the library urdfpy

File: pkg/urdf/robot.urdf (robot description, URDF)
Before this commit: robot Assemblage robot.SLDASM, 13 links, 12 joints
Links:
- link arm_to_forearm_1: geometry collision mesh filename=../../pkg/meshes/arm_to_forearm_1.STL; visual mesh filename=../../pkg/meshes/arm_to_forearm_1.STL
- link arm_to_forearm_2: geometry collision mesh filename=../../pkg/meshes/arm_to_forearm_2.STL; visual mesh filename=../../pkg/meshes/arm_to_forearm_2.STL
- link arm_to_forearm_3: geometry collision mesh filename=../../pkg/meshes/arm_to_forearm_3.STL; visual mesh filename=../../pkg/meshes/arm_to_forearm_3.STL
- link base_link: geometry collision mesh filename=../../pkg/meshes/base_link.STL; visual mesh filename=../../pkg/meshes/base_link.STL
- link forearm_to_hand_1: geometry collision mesh filename=../../pkg/meshes/forearm_to_hand_1.STL; visual mesh filename=../../pkg/meshes/forearm_to_hand_1.STL
- link forearm_to_hand_2: geometry collision mesh filename=../../pkg/meshes/forearm_to_hand_2.STL; visual mesh filename=../../pkg/meshes/forearm_to_hand_2.STL
- link forearm_to_hand_3: geometry collision mesh filename=../../pkg/meshes/forearm_to_hand_3.STL; visual mesh filename=../../pkg/meshes/forearm_to_hand_3.STL
- link motor_to_arm_1: geometry collision mesh filename=../../pkg/meshes/motor_to_arm_1.STL; visual mesh filename=../../pkg/meshes/motor_to_arm_1.STL
- link motor_to_arm_2: geometry collision mesh filename=../../pkg/meshes/motor_to_arm_2.STL; visual mesh filename=../../pkg/meshes/motor_to_arm_2.STL
- link motor_to_arm_3: geometry collision mesh filename=../../pkg/meshes/motor_to_arm_3.STL; visual mesh filename=../../pkg/meshes/motor_to_arm_3.STL
- link motorlink1: geometry collision mesh filename=../../pkg/meshes/motorlink1.STL; visual mesh filename=../../pkg/meshes/motorlink1.STL
- link motorlink2: geometry collision mesh filename=../../pkg/meshes/motorlink2.STL; visual mesh filename=../../pkg/meshes/motorlink2.STL
- link motorlink3: geometry collision mesh filename=../../pkg/meshes/motorlink3.STL; visual mesh filename=../../pkg/meshes/motorlink3.STL
